Commit message: feat: atualizando plug in

File: urdf/rosbot3.xacro (robot description, xacro)
@@ -8,23 +8,14 @@
   <xacro:include filename="$(find rosbot3_description)/urdf/rosbot3.xacro"/>
   <xacro:include filename="$(find ros_commons)/urdf/gazebo.xacro"/>
-  <xacro:macro
-    name="add_controller"
-    params="
-      position
-    "
-  >
-    <xacro:differential_controller
-      name="wheels_${position}"
-      left_joint="joint_wheel_${position}_left"
-      right_joint="joint_wheel_${position}_right"
-      wheel_separation="${wheel_separation}"
-      wheel_diameter="${wheel_diameter}"
-    />
-  </xacro:macro>
-  <!-- Controllers for both axles -->
-  <xacro:add_controller position="front"/>
-  <xacro:add_controller position="rear"/>
-  <!-- Removing friction for front axle-->
-  <xacro:remove_friction position="front"/>
+  <xacro:skid_steer_controller
+    name="skid_steer_controller"
+    front_left_joint="joint_wheel_front_left"
+    front_right_joint="joint_wheel_front_right"
+    rear_left_joint="joint_wheel_rear_left"
+    rear_right_joint="joint_wheel_rear_right"
+    wheel_separation="${wheel_separation}"
+    wheel_diameter="${wheel_diameter}"
+    publish_odom="true"
+  />
   <xacro:depth_camera name="camera_front"/>
   <xacro:lidar_2d name="laser"/>

Commit message: feat: retornando plug in

File: urdf/rosbot3.xacro (robot description, xacro)
@@ -8,14 +8,25 @@
   <xacro:include filename="$(find rosbot3_description)/urdf/rosbot3.xacro"/>
   <xacro:include filename="$(find ros_commons)/urdf/gazebo.xacro"/>
-  <xacro:skid_steer_controller
-    name="skid_steer_controller"
-    front_left_joint="joint_wheel_front_left"
-    front_right_joint="joint_wheel_front_right"
-    rear_left_joint="joint_wheel_rear_left"
-    rear_right_joint="joint_wheel_rear_right"
-    wheel_separation="${wheel_separation}"
-    wheel_diameter="${wheel_diameter}"
-    publish_odom="true"
-  />
+  <xacro:macro
+    name="add_controller"
+    params="
+      position
+      publish_odom:=false
+    "
+  >
+    <xacro:differential_controller
+      name="wheels_${position}"
+      left_joint="joint_wheel_${position}_left"
+      right_joint="joint_wheel_${position}_right"
+      wheel_separation="${wheel_separation}"
+      wheel_diameter="${wheel_diameter}"
+      publish_odom="${publish_odom}"
+    />
+  </xacro:macro>
+  <!-- Controllers for both axles -->
+  <xacro:add_controller position="front"/>
+  <xacro:add_controller position="rear" publish_odom="true"/>
+  <!-- Removing friction for front axle-->
+  <xacro:remove_friction position="front"/>
   <xacro:depth_camera name="camera_front"/>
   <xacro:lidar_2d name="laser"/>

Commit message: Revert "feat: retornando plug in"
This reverts commit ae5e2c53318f3b0597be38095d978d3672bb4e2a.

File: urdf/rosbot3.xacro (robot description, xacro)
@@ -8,25 +8,14 @@
   <xacro:include filename="$(find rosbot3_description)/urdf/rosbot3.xacro"/>
   <xacro:include filename="$(find ros_commons)/urdf/gazebo.xacro"/>
-  <xacro:macro
-    name="add_controller"
-    params="
-      position
-      publish_odom:=false
-    "
-  >
-    <xacro:differential_controller
-      name="wheels_${position}"
-      left_joint="joint_wheel_${position}_left"
-      right_joint="joint_wheel_${position}_right"
-      wheel_separation="${wheel_separation}"
-      wheel_diameter="${wheel_diameter}"
-      publish_odom="${publish_odom}"
-    />
-  </xacro:macro>
-  <!-- Controllers for both axles -->
-  <xacro:add_controller position="front"/>
-  <xacro:add_controller position="rear" publish_odom="true"/>
-  <!-- Removing friction for front axle-->
-  <xacro:remove_friction position="front"/>
+  <xacro:skid_steer_controller
+    name="skid_steer_controller"
+    front_left_joint="joint_wheel_front_left"
+    front_right_joint="joint_wheel_front_right"
+    rear_left_joint="joint_wheel_rear_left"
+    rear_right_joint="joint_wheel_rear_right"
+    wheel_separation="${wheel_separation}"
+    wheel_diameter="${wheel_diameter}"
+    publish_odom="true"
+  />
   <xacro:depth_camera name="camera_front"/>
   <xacro:lidar_2d name="laser"/>

Commit message: feat: adequando o diff drive ao skid steer

File: urdf/rosbot3.xacro (robot description, xacro)
@@ -8,25 +8,17 @@
   <xacro:include filename="$(find rosbot3_description)/urdf/rosbot3.xacro"/>
   <xacro:include filename="$(find ros_commons)/urdf/gazebo.xacro"/>
-  <xacro:macro
-    name="add_controller"
-    params="
-      position
-      publish_odom:=false
-    "
-  >
-    <xacro:differential_controller
-      name="wheels_${position}"
-      left_joint="joint_wheel_${position}_left"
-      right_joint="joint_wheel_${position}_right"
-      wheel_separation="${wheel_separation}"
-      wheel_diameter="${wheel_diameter}"
-      publish_odom="${publish_odom}"
-    />
-  </xacro:macro>
-  <!-- Controllers for both axles -->
-  <xacro:add_controller position="front"/>
-  <xacro:add_controller position="rear" publish_odom="true"/>
-  <!-- Removing friction for front axle-->
-  <xacro:remove_friction position="front"/>
+<!-- New controller for skid steer -->
+  <xacro:skid_steer_controller
+    name="skid_steer_base_controller"
+    front_left_joint="joint_wheel_front_left"
+    front_right_joint="joint_wheel_front_right"
+    rear_left_joint="joint_wheel_rear_left"
+    rear_right_joint="joint_wheel_rear_right"
+    front_wheel_separation="0.5"
+    rear_wheel_separation="0.5"
+    front_wheel_diameter="0.15"
+    rear_wheel_diameter="0.15"
+    publish_odom="true"
+  />
   <xacro:depth_camera name="camera_front"/>
   <xacro:lidar_2d name="laser"/>
